File: Z80/Z80_PCB_Design/Z80_CPU/Z80_CPU.sch (KiCad schematic (older format))
At the start: 5 parts

Commit message: Z80 retro CPU design with PSoC Glue Logic
Parts:
- removed J?: Conn_02x02_Odd_Even, symbol Connector_Generic:Conn_02x02_Odd_Even
- removed R? (x2): 10K, symbol Device:R_Small
- added U?: Z8430, symbol Easy_Z80:my_components_Z84C30
- added U?: Z8470, symbol Easy_Z80:my_components_Z84C40
- added U?: CY8C5888AXI-LP096, MODULE, symbol LandBoards_Semis:CY8C5888AXI-LP096
- added U? (x2): HM62256BLP-7, DIP28, symbol RC6502_Apple_1_SBC:HM62256BLP-7
- added U? (x2): Z8420, Package_DIP:DIP-40_W15.24mm, symbol z80_Interface:Z8420
- U?: symbol Zilog:Z80CPU -> Z80_CPU-rescue:Z80CPU-Zilog
Connections:
- net labels added: CPUCLK, EEPA13, EEPA14, SRAMA13, SRAMA14, ~CPURST, ~MEMRD, ~MEMWR, ~SRAMCS0, ~SRAMCS1
- net labels removed: ~EEOE, ~EEWR
- wire segments 83 -> 189
Other:
- moved on the sheet: U?

Commit message: Moved around KiCad libraries. May need to link to new libraries.
Parts:
- U?: symbol Easy_Z80:my_components_Z84C30 -> Z80_CPU-rescue:my_components_Z84C30-Easy_Z80
- U?: symbol Easy_Z80:my_components_Z84C40 -> Z80_CPU-rescue:my_components_Z84C40-Easy_Z80
- U? (x2): symbol RC6502_Apple_1_SBC:HM62256BLP-7 -> Z80_CPU-rescue:HM62256BLP-7-RC6502_Apple_1_SBC
- U? (x2): symbol z80_Interface:Z8420 -> Z80_CPU-rescue:Z8420-z80_Interface
Connections:
- net labels added: RFSH, ~BUSACK, ~BUSRQ, ~CPURD, ~CPUWR, ~HALT, ~INT, ~IORQ, ~M1, ~MREQ, ~NMI, ~WAIT
- wire segments 189 -> 197
Changed lines of the file:
@@
 ~EECS
 $Comp
-L Easy_Z80:my_components_Z84C30 U?
+L Z80_CPU-rescue:my_components_Z84C30-Easy_Z80 U?
 U 1 1 5D72F299
 P 6650 5800
@@
 $EndComp
 $Comp
-L Easy_Z80:my_components_Z84C40 U?
+L Z80_CPU-rescue:my_components_Z84C40-Easy_Z80 U?
 U 1 1 5D72F39B
 P 2300 6000
@@
 ~MEMRD
 $Comp
-L RC6502_Apple_1_SBC:HM62256BLP-7 U?
+L Z80_CPU-rescue:HM62256BLP-7-RC6502_Apple_1_SBC U?
 U 1 1 5D7CD253
 P 7500 1950
@@
 $EndComp
 $Comp
-L RC6502_Apple_1_SBC:HM62256BLP-7 U?
+L Z80_CPU-rescue:HM62256BLP-7-RC6502_Apple_1_SBC U?
 U 1 1 5D7CD35B
 P 10050 1950
@@
 CPUCLK
 $Comp
-L z80_Interface:Z8420 U?
+L Z80_CPU-rescue:Z8420-z80_Interface U?
 U 1 1 5D9335AC
 P 2250 9050
@@
 $EndComp
 $Comp
-L z80_Interface:Z8420 U?
+L Z80_CPU-rescue:Z8420-z80_Interface U?
 U 1 1 5D933648
 P 6700 9050
@@
 	1    0    0    -1
 $EndComp
+Text Label 900  1800 0    50   ~ 0
+~NMI
+Text Label 900  1900 0    50   ~ 0
+~INT
+Text Label 15150 4050 0    50   ~ 0
+~NMI
+Text Label 15150 4150 0    50   ~ 0
+~INT
+Text Label 900  2200 0    50   ~ 0
+~M1
+Text Label 900  2300 0    50   ~ 0
+RFSH
+Text Label 900  2400 0    50   ~ 0
+~WAIT
+Text Label 900  2500 0    50   ~ 0
+~HALT
+Text Label 900  2900 0    50   ~ 0
+~CPURD
+Text Label 900  3000 0    50   ~ 0
+~CPUWR
+Text Label 900  3100 0    50   ~ 0
+~MREQ
+Text Label 900  3200 0    50   ~ 0
+~IORQ
+Text Label 900  3500 0    50   ~ 0
+~BUSRQ
+Text Label 900  3600 0    50   ~ 0
+~BUSACK
+Text Label 15150 4250 0    50   ~ 0
+~M1
+Text Label 15150 4350 0    50   ~ 0
+RFSH
+Text Label 15150 4450 0    50   ~ 0
+~WAIT
+Text Label 15150 4550 0    50   ~ 0
+~HALT
+Text Label 15150 4750 0    50   ~ 0
+~CPURD
+Text Label 15150 4850 0    50   ~ 0
+~CPUWR
+Text Label 15150 4950 0    50   ~ 0
+~MREQ
+Text Label 15150 5050 0    50   ~ 0
+~IORQ
+Text Label 15150 5150 0    50   ~ 0
+~BUSRQ
+Text Label 15150 5250 0    50   ~ 0
+~BUSACK
+Wire Wire Line
+	14950 4750 15550 4750
+Wire Wire Line
+	14950 4850 15550 4850
+Wire Wire Line
+	14950 4950 15550 4950
+Wire Wire Line
+	14950 5050 15550 5050
+Wire Wire Line
+	14950 5150 15550 5150
+Wire Wire Line
+	14950 5250 15550 5250
+Wire Wire Line
+	14950 5350 15550 5350
+Wire Wire Line
+	14950 5450 15550 5450
 $EndSCHEMATC

Commit message: More Z80 stuff
Parts:
- added C? (x2): 10pF, symbol Device:C
- added D?: LED_Small_ALT, symbol Device:LED_Small_ALT
- added R?: R, symbol Device:R
- added Y?: 32.768KHz, symbol Device:Crystal
- U?: value CY8C5888AXI-LP096 -> CY8C5267AXI-LP051
Connections:
- net labels added: ~CTCCS, ~DARTCS, ~PIOCS1, ~PIOCS2
- wire segments 197 -> 218
Changed lines of the file:
@@
 P 13750 5700
 F 0 "U?" H 14600 8450 50  0000 C CNN
-F 1 "CY8C5888AXI-LP096" H 14600 2950 50  0000 C CNN
+F 1 "CY8C5267AXI-LP051" H 14600 2950 50  0000 C CNN
 F 2 "MODULE" H 13750 5700 50  0001 C CNN
 F 3 "DOCUMENTATION" H 13650 3450 50  0001 C CNN
@@
 	14950 5250 15550 5250
 Wire Wire Line
-	14950 5350 15550 5350
+	14950 5350 16100 5350
 Wire Wire Line
 	14950 5450 15550 5450
+$Comp
+L Device:LED_Small_ALT D?
+U 1 1 5D7D31EE
+P 16100 4800
+F 0 "D?" V 16146 4732 50  0000 R CNN
+F 1 "LED_Small_ALT" V 16055 4732 50  0000 R CNN
+F 2 "" V 16100 4800 50  0001 C CNN
+F 3 "~" V 16100 4800 50  0001 C CNN
+	1    16100 4800
+	0    -1   -1   0
+$EndComp
+$Comp
+L Device:R R?
+U 1 1 5D7D3281
+P 16100 5100
+F 0 "R?" H 16170 5146 50  0000 L CNN
+F 1 "R" H 16170 5055 50  0000 L CNN
+F 2 "" V 16030 5100 50  0001 C CNN
+F 3 "~" H 16100 5100 50  0001 C CNN
+	1    16100 5100
+	1    0    0    -1
+$EndComp
+Wire Wire Line
+	16100 4900 16100 4950
+Wire Wire Line
+	16100 5250 16100 5350
+Wire Wire Line
+	16100 4700 16100 4550
+$Comp
+L power:+5V #PWR?
+U 1 1 5D80D2C6
+P 16100 4550
+F 0 "#PWR?" H 16100 4400 50  0001 C CNN
+F 1 "+5V" H 16115 4723 50  0000 C CNN
+F 2 "" H 16100 4550 50  0001 C CNN
+F 3 "" H 16100 4550 50  0001 C CNN
+	1    16100 4550
+	1    0    0    -1
+$EndComp
+Wire Wire Line
+	1000 5800 1600 5800
+Text Label 1100 5800 0    50   ~ 0
+~DARTCS
+Wire Wire Line
+	5350 5800 5950 5800
+Text Label 5450 5800 0    50   ~ 0
+~CTCCS
+Wire Wire Line
+	1150 9150 1750 9150
+Text Label 1250 9150 0    50   ~ 0
+~PIOCS1
+Wire Wire Line
+	5600 9150 6200 9150
+Text Label 5700 9150 0    50   ~ 0
+~PIOCS2
+$Comp
+L Device:Crystal Y?
+U 1 1 5D849E1F
+P 16000 6900
+F 0 "Y?" V 15954 7031 50  0000 L CNN
+F 1 "32.768KHz" V 16045 7031 50  0000 L CNN
+F 2 "" H 16000 6900 50  0001 C CNN
+F 3 "~" H 16000 6900 50  0001 C CNN
+	1    16000 6900
+	0    1    1    0
+$EndComp
+Wire Wire Line
+	14950 6950 15350 6950
+Wire Wire Line
+	15350 6950 15350 6700
+Wire Wire Line
+	15350 6700 16000 6700
+Wire Wire Line
+	16000 6700 16000 6750
+Wire Wire Line
+	14950 7050 15350 7050
+Wire Wire Line
+	15350 7050 15350 7100
+Wire Wire Line
+	15350 7100 16000 7100
+Wire Wire Line
+	16000 7100 16000 7050
+$Comp
+L Device:C C?
+U 1 1 5D87A0E7
+P 16000 6500
+F 0 "C?" H 16115 6546 50  0000 L CNN
+F 1 "10pF" H 16115 6455 50  0000 L CNN
+F 2 "" H 16038 6350 50  0001 C CNN
+F 3 "~" H 16000 6500 50  0001 C CNN
+	1    16000 6500
+	1    0    0    -1
+$EndComp
+$Comp
+L Device:C C?
+U 1 1 5D87A16D
+P 16000 7300
+F 0 "C?" H 16115 7346 50  0000 L CNN
+F 1 "10pF" H 16115 7255 50  0000 L CNN
+F 2 "" H 16038 7150 50  0001 C CNN
+F 3 "~" H 16000 7300 50  0001 C CNN
+	1    16000 7300
+	1    0    0    -1
+$EndComp
+Wire Wire Line
+	16000 6650 16000 6700
+Connection ~ 16000 6700
+Wire Wire Line
+	16000 7100 16000 7150
+Connection ~ 16000 7100
+Wire Wire Line
+	16000 7450 16000 7500
+Wire Wire Line
+	16000 6350 16000 6300
+Wire Wire Line
+	16000 6300 16400 6300
+Wire Wire Line
+	16400 6300 16400 6400
+$Comp
+L power:GND #PWR?
+U 1 1 5D8BAB50
+P 16400 6400
+F 0 "#PWR?" H 16400 6150 50  0001 C CNN
+F 1 "GND" H 16405 6227 50  0000 C CNN
+F 2 "" H 16400 6400 50  0001 C CNN
+F 3 "" H 16400 6400 50  0001 C CNN
+	1    16400 6400
+	1    0    0    -1
+$EndComp
+$Comp
+L power:GND #PWR?
+U 1 1 5D8BABF5
+P 16000 7500
+F 0 "#PWR?" H 16000 7250 50  0001 C CNN
+F 1 "GND" H 16005 7327 50  0000 C CNN
+F 2 "" H 16000 7500 50  0001 C CNN
+F 3 "" H 16000 7500 50  0001 C CNN
+	1    16000 7500
+	1    0    0    -1
+$EndComp
 $EndSCHEMATC

Commit message: Did more Z80 retro stuff
Parts:
- added BRD?: FTDI-Slave, Connector_PinHeader_2.54mm:PinHeader_1x06_P2.54mm_Vertical, symbol LandBoards_Cards:FTDI-Slave
- added BT?: Battery_Cell, symbol Device:Battery_Cell
- added C? (x13): 0.1uF, Capacitor_SMD:C_0805_2012Metric_Pad1.15x1.40mm_HandSolder, symbol Device:C_Small
- added C? (x4): 1uF, symbol Device:C_Small
- added J?: Conn_01x04, symbol Connector_Generic:Conn_01x04
- added J?: USB_B, symbol Connector:USB_B
- added J? (x4): Conn_01x08, symbol Connector_Generic:Conn_01x08
- added L?: ChipInd, symbol Device:L_Small
- added R? (x3): 3.9K, Resistor_SMD:R_0805_2012Metric_Pad1.15x1.40mm_HandSolder, symbol Device:R
- added R? (x2): 22, symbol Device:R_Small
- added R?: 3.9K, symbol Device:R
- added U?: 4.9152 MHz, symbol LandBoards_Semis:OSC
- R?: value R -> 330
- U? (x2): footprint DIP28 -> Package_DIP:DIP-28_W15.24mm
Connections:
- net labels added: +3.3V, CTCINT_O, DINT_O, PIO1INT_O, SER_D2F1, SER_D2P, SER_F2D1, SER_P2D, S_D_CTS, S_D_CTS2, S_D_RTS, S_D_RTS1, S_D_RTS2, UARTCLK, USB-DM, USB-DP
- wire segments 218 -> 453
- no-connect marks 0 -> 2
Other:
- note added: "PSoC \nDownload\nConnector"
- moved on the sheet: C?, D?, R?, U?, Y?

Commit message: FPGA build of 9 chip Z80
Parts:
- BRD?: symbol LandBoards_Cards:FTDI-Slave -> Z80_CPU-rescue:FTDI-Slave-LandBoards_Cards
- J?: symbol Connector:USB_B -> Z80_CPU-rescue:USB_B-Connector
Changed lines of the file:
@@
 U 1 1 5D72F299
 P 5550 5600
-F 0 "U?" H 5550 6838 60  0000 C CNN
-F 1 "Z8430" H 5550 6732 60  0000 C CNN
+F 0 "U?" H 5700 6700 60  0000 C CNN
+F 1 "Z8430" H 5800 4550 60  0000 C CNN
 F 2 "" H 5550 5300 60  0000 C CNN
 F 3 "" H 5550 5300 60  0000 C CNN
@@
 USB-DP
 $Comp
-L Connector:USB_B J?
+L Z80_CPU-rescue:USB_B-Connector J?
 U 1 1 5DCE587A
 P 14050 7900
@@
 SER_D2F1
 $Comp
-L LandBoards_Cards:FTDI-Slave BRD?
+L Z80_CPU-rescue:FTDI-Slave-LandBoards_Cards BRD?
 U 1 1 5E25204B
 P 4500 7200

Commit message: Z80 3-chip design
Parts:
- BT1: renamed from BT?; footprint (none) -> Battery:BatteryHolder_Keystone_1060_1x2032
- C2, C3, C4, C5, C7, C8: renamed from C?; footprint (none) -> Capacitor_SMD:C_0805_2012Metric_Pad1.15x1.40mm_HandSolder
- D1: renamed from D?; footprint (none) -> LED_THT:LED_D3.0mm_Horizontal_O1.27mm_Z2.0mm
- J1, J2, J3, J4: renamed from J?; footprint (none) -> Connector_PinHeader_2.54mm:PinHeader_1x08_P2.54mm_Vertical
- J5: renamed from J?; footprint (none) -> Connector_PinHeader_2.54mm:PinHeader_1x04_P2.54mm_Vertical
- J6: renamed from J?; footprint (none) -> Connector_USB:USB_B_OST_USB-B1HSxx_Horizontal
- L1: renamed from L?; footprint (none) -> Inductor_SMD:L_0805_2012Metric_Pad1.15x1.40mm_HandSolder
- R3, R5, R6, R7: renamed from R?; footprint (none) -> Resistor_SMD:R_0805_2012Metric_Pad1.15x1.40mm_HandSolder
- U10: renamed from U?; footprint (none) -> Oscillator:Oscillator_DIP-14
- U3: renamed from U?; footprint (none) -> Package_DIP:DIP-40_W15.24mm
- U5: renamed from U?; footprint (none) -> Package_DIP:DIP-28_W15.24mm
- U8: renamed from U?; footprint MODULE -> Package_QFP:TQFP-100_14x14mm_P0.5mm
- Y1: renamed from Y?; footprint (none) -> Crystal:Crystal_HC18-U_Horizontal
- gave numbers to parts that had none: 23
Connections:
- net labels added: S_D_CTS1, ~IOCS, ~WRMRST
- net labels removed: S_D_RTS
- wire segments 453 -> 458
