File: Z80/Z80_PCB_Design/Z80_CPU-3ICs/Z80_CPU.sch (KiCad schematic (older format))
At the start: 37 parts, among them J1 USB_B, U1 Z80CPU, U2 AS6C4008-55PCN, U3 4.9152 MHz, U4 CY8C5267AXI-LP051, Y1 32.768KHz

Commit message: Z80 Front Panel Design
Parts:
- removed U2: AS6C4008-55PCN, Package_DIP:DIP-32_W15.24mm, symbol Easy_Z80:AS6C4008
- added U2: my_components_AS6C4008_PWR, Package_DIP:DIP-32_W15.24mm, symbol Easy_Z80:my_components_AS6C4008_PWR
Connections:
- net labels added: SRAMA11, SRAMA12
- wire segments 285 -> 287
Changed lines of the file:
@@
 CPUA10
 Text Label 4050 7150 0    50   ~ 0
-CPUA11
+SRAMA11
 Text Label 4050 7250 0    50   ~ 0
-CPUA12
+SRAMA12
 Text Label 4050 7350 0    50   ~ 0
 SRAMA13
@@
 L power:+5V #PWR0102
 U 1 1 5DDBEE11
-P 5150 5750
-F 0 "#PWR0102" H 5150 5600 50  0001 C CNN
-F 1 "+5V" H 5165 5923 50  0000 C CNN
-F 2 "" H 5150 5750 50  0001 C CNN
-F 3 "" H 5150 5750 50  0001 C CNN
-	1    5150 5750
-	1    0    0    -1
-$EndComp
-Wire Wire Line
-	5150 5800 5150 5750
+P 5750 8200
+F 0 "#PWR0102" H 5750 8050 50  0001 C CNN
+F 1 "+5V" H 5765 8373 50  0000 C CNN
+F 2 "" H 5750 8200 50  0001 C CNN
+F 3 "" H 5750 8200 50  0001 C CNN
+	1    5750 8200
+	1    0    0    -1
+$EndComp
+Wire Wire Line
+	5750 8250 5750 8200
 $Comp
 L power:GND #PWR0104
@@
 Wire Wire Line
 	13650 4550 13750 4550
-$Comp
-L Easy_Z80:AS6C4008 U2
-U 1 1 5DFD81C3
-P 5150 7150
-F 0 "U2" H 5400 8400 60  0000 C CNN
-F 1 "AS6C4008-55PCN" H 5650 5900 60  0000 C CNN
-F 2 "Package_DIP:DIP-32_W15.24mm" H 6000 5800 60  0000 C CNN
-F 3 "" H 5150 7150 60  0000 C CNN
-	1    5150 7150
-	1    0    0    -1
-$EndComp
 Wire Wire Line
 	8600 3850 7650 3850
@@
 	13700 3400 13700 3500
 $Comp
-L power:GND #PWR?
+L power:GND #PWR0119
 U 1 1 5D8B3EF1
 P 13700 3500
-F 0 "#PWR?" H 13700 3250 50  0001 C CNN
+F 0 "#PWR0119" H 13700 3250 50  0001 C CNN
 F 1 "GND" H 13705 3327 50  0000 C CNN
 F 2 "" H 13700 3500 50  0001 C CNN
@@
 	13700 3400 13800 3400
 $Comp
-L power:+5V #PWR?
+L power:+5V #PWR0120
 U 1 1 5D8FE114
 P 13700 2700
-F 0 "#PWR?" H 13700 2550 50  0001 C CNN
+F 0 "#PWR0120" H 13700 2550 50  0001 C CNN
 F 1 "+5V" H 13715 2873 50  0000 C CNN
 F 2 "" H 13700 2700 50  0001 C CNN
@@
 	1    0    0    -1
 $EndComp
+Wire Wire Line
+	8000 5350 8600 5350
+Wire Wire Line
+	8000 5450 8600 5450
+Text Label 8100 5450 0    50   ~ 0
+SRAMA11
+Text Label 8100 5350 0    50   ~ 0
+SRAMA12
+$Comp
+L Easy_Z80:my_components_AS6C4008_PWR U2
+U 1 1 5D8EC51F
+P 5150 7150
+F 0 "U2" H 5150 8643 60  0000 C CNN
+F 1 "my_components_AS6C4008_PWR" H 5150 8537 60  0000 C CNN
+F 2 "Package_DIP:DIP-32_W15.24mm" H 5150 8431 60  0000 C CNN
+F 3 "" H 5150 7150 60  0000 C CNN
+	1    5150 7150
+	1    0    0    -1
+$EndComp

Commit message: Front panel design
Parts:
- added J2, J3: Conn_01x10, Connector_PinHeader_2.54mm:PinHeader_1x10_P2.54mm_Vertical, symbol Connector_Generic:Conn_01x10
- added U5: MCP23017_SP, Package_DIP:DIP-28_W7.62mm, symbol Interface_Expansion:MCP23017_SP
- U2: symbol Easy_Z80:my_components_AS6C4008_PWR -> Z80_CPU-rescue:my_components_AS6C4008_PWR-Easy_Z80
Connections:
- wire segments 287 -> 328
Other:
- moved on the sheet: BT1, C1, C2, C3, C4, C5, C7, C8, D1, H1, H2, H3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

Commit message: z80 cpu legends
Connections:
- net labels added: GPA0, GPA7, GPB0, GPB7
Other:
- moved on the sheet: J2, J3
Changed lines of the file:
@@
 L Connector_Generic:Conn_01x10 J2
 U 1 1 5D8C51E7
-P 4050 6750
-F 0 "J2" H 4130 6742 50  0000 L CNN
-F 1 "Conn_01x10" H 4130 6651 50  0000 L CNN
-F 2 "Connector_PinHeader_2.54mm:PinHeader_1x10_P2.54mm_Vertical" H 4050 6750 50  0001 C CNN
-F 3 "~" H 4050 6750 50  0001 C CNN
-	1    4050 6750
-	1    0    0    -1
+P 4300 6850
+F 0 "J2" H 4250 6250 50  0000 L CNN
+F 1 "Conn_01x10" H 4250 6200 50  0000 L CNN
+F 2 "Connector_PinHeader_2.54mm:PinHeader_1x10_P2.54mm_Vertical" H 4500 7700 30  0000 C CNN
+F 3 "~" H 4300 6850 50  0001 C CNN
+	1    4300 6850
+	1    0    0    1
 $EndComp
 $Comp
 L Connector_Generic:Conn_01x10 J3
 U 1 1 5D8DE613
-P 4450 7650
-F 0 "J3" H 4400 8150 50  0000 L CNN
-F 1 "Conn_01x10" H 4100 7050 50  0000 L CNN
-F 2 "Connector_PinHeader_2.54mm:PinHeader_1x10_P2.54mm_Vertical" H 4450 7650 50  0000 C CNN
-F 3 "~" H 4450 7650 50  0001 C CNN
-	1    4450 7650
+P 4750 7650
+F 0 "J3" H 4700 8150 50  0000 L CNN
+F 1 "Conn_01x10" H 4400 7050 50  0000 L CNN
+F 2 "Connector_PinHeader_2.54mm:PinHeader_1x10_P2.54mm_Vertical" H 4750 7000 30  0000 C CNN
+F 3 "~" H 4750 7650 50  0001 C CNN
+	1    4750 7650
 	1    0    0    -1
 $EndComp
 Wire Wire Line
-	3700 6450 3850 6450
+	3700 6450 4100 6450
 Wire Wire Line
-	3850 6550 3700 6550
+	4100 6550 3700 6550
 Wire Wire Line
-	3700 6650 3850 6650
+	3700 6650 4100 6650
 Wire Wire Line
-	3700 6750 3850 6750
+	3700 6750 4100 6750
 Wire Wire Line
-	3700 6850 3850 6850
+	3700 6850 4100 6850
 Wire Wire Line
-	3700 6950 3850 6950
+	3700 6950 4100 6950
 Wire Wire Line
-	3700 7050 3850 7050
+	3700 7050 4100 7050
 Wire Wire Line
-	3700 7150 3850 7150
+	3700 7150 4100 7150
 Wire Wire Line
-	3700 7350 4250 7350
+	3700 7350 4550 7350
 Wire Wire Line
-	3700 7450 4250 7450
+	3700 7450 4550 7450
 Wire Wire Line
-	3700 7550 4250 7550
+	3700 7550 4550 7550
 Wire Wire Line
-	3700 7650 4250 7650
+	3700 7650 4550 7650
 Wire Wire Line
-	3700 7750 4250 7750
+	3700 7750 4550 7750
 Wire Wire Line
-	3700 7850 4250 7850
+	3700 7850 4550 7850
 Wire Wire Line
-	3700 7950 4250 7950
+	3700 7950 4550 7950
 Wire Wire Line
-	3700 8050 4250 8050
+	3700 8050 4550 8050
 Wire Wire Line
-	3850 7250 3800 7250
-Wire Wire Line
-	3800 7250 3800 8150
-Wire Wire Line
-	3800 8150 4250 8150
-Wire Wire Line
-	3800 8150 3800 8450
+	4100 7250 3800 7250
 Wire Wire Line
 	3800 8450 3000 8450
 Wire Wire Line
 	3000 8450 3000 8350
-Connection ~ 3800 8150
 Wire Wire Line
 	3000 8450 3000 8550
@@
 $EndComp
 Wire Wire Line
-	4250 7250 4150 7250
+	4400 6100 3750 6100
 Wire Wire Line
-	4150 7250 4150 6250
+	3750 6100 3750 6350
 Wire Wire Line
-	4150 6250 3750 6250
-Wire Wire Line
-	3750 6250 3750 6350
-Wire Wire Line
-	3750 6350 3850 6350
+	3750 6350 4100 6350
 Wire Wire Line
 	3000 6150 3000 6100
 Wire Wire Line
 	3000 6100 3750 6100
-Wire Wire Line
-	3750 6100 3750 6250
-Connection ~ 3750 6250
+Connection ~ 3750 6100
 Wire Wire Line
 	3000 6100 3000 6000
@@
 Text Label 1800 6550 0    50   ~ 0
 SCL
+Text Label 3800 6450 0    50   ~ 0
+GPB0
+Text Label 3800 7150 0    50   ~ 0
+GPB7
+Text Label 3900 7350 0    50   ~ 0
+GPA0
+Text Label 3900 8050 0    50   ~ 0
+GPA7
+Wire Wire Line
+	3800 7250 3800 8450
+Wire Wire Line
+	4550 7250 4500 7250
+Wire Wire Line
+	4500 7250 4500 8450
+Wire Wire Line
+	4500 8450 3800 8450
+Connection ~ 3800 8450
+Wire Wire Line
+	4550 8150 4400 8150
+Wire Wire Line
+	4400 6100 4400 8150
 $EndSCHEMATC

Commit message: Added I2C interface to Z80 CPU
Parts:
- removed H1: Conn_01x04, Connector_PinHeader_2.54mm:PinHeader_1x04_P2.54mm_Vertical, symbol Connector_Generic:Conn_01x04
- removed J2, J3: Conn_01x10, Connector_PinHeader_2.54mm:PinHeader_1x10_P2.54mm_Vertical, symbol Connector_Generic:Conn_01x10
- removed U2: my_components_AS6C4008_PWR, Package_DIP:DIP-32_W15.24mm, symbol Z80_CPU-rescue:my_components_AS6C4008_PWR-Easy_Z80
- added H1: Conn_01x05, Connector_PinHeader_2.54mm:PinHeader_1x05_P2.54mm_Vertical, symbol Connector_Generic:Conn_01x05
- added J2, J3: Conn_01x12, Connector_PinHeader_2.54mm:PinHeader_1x12_P2.54mm_Vertical, symbol Connector_Generic:Conn_01x12
- added U2: AS6C4008, symbol Z80_CPU-rescue:AS6C4008
- U5: symbol Interface_Expansion:MCP23017_SP -> Z80_CPU-rescue:MCP23017_SP-Interface_Expansion
Connections:
- net labels added: GPA1, GPA2, GPA3, GPA4, GPA5, GPA6, GPB1, GPB2, GPB3, GPB4, GPB5, GPB6, ~I2CINT
- wire segments 328 -> 346
- no-connect marks 10 -> 14
Other:
- note added: "(VIA)"
- moved on the sheet: U5

Commit message: z80
Parts:
- added C16: 10pF, Capacitor_SMD:C_0805_2012Metric_Pad1.15x1.40mm_HandSolder, symbol Device:C
- added J4: Conn_01x02, Connector_PinHeader_2.54mm:PinHeader_1x02_P2.54mm_Vertical, symbol Connector_Generic:Conn_01x02
- added R1, R2, R3, R8, R9: 2.2K, Resistor_SMD:R_0805_2012Metric_Pad1.15x1.40mm_HandSolder, symbol Device:R
Connections:
- net labels added: DAC_OUT
- wire segments 346 -> 370
- no-connect marks 14 -> 12
Changed lines of the file:
@@
 Text Label 9450 5300 0    50   ~ 0
 SRAMA14
-Wire Wire Line
-	14500 4500 15100 4500
-Wire Wire Line
-	14500 4400 15100 4400
 Text Label 12650 5100 0    50   ~ 0
 SDA
@@
 NoConn ~ 12500 7300
 NoConn ~ 12500 7400
-NoConn ~ 12500 6000
 $Comp
 L power:+5V #PWR0118
@@
 	1    0    0    1
 $EndComp
-Wire Wire Line
-	15100 4300 14500 4300
 Text Label 14600 4300 0    50   ~ 0
 ~I2CINT
@@
 NoConn ~ 12500 4900
 NoConn ~ 12500 5000
-NoConn ~ 12500 5400
 NoConn ~ 12500 5500
-Text Notes 12550 5400 0    50   ~ 0
-(VIA)
 Text Notes 12550 5500 0    50   ~ 0
 (VIA)
@@
 	2050 5400 2050 5500
 Connection ~ 3200 4150
+$Comp
+L Device:R R3
+U 1 1 5D8E849B
+P 14400 4050
+F 0 "R3" H 14470 4096 50  0000 L CNN
+F 1 "2.2K" H 14470 4005 50  0000 L CNN
+F 2 "Resistor_SMD:R_0805_2012Metric_Pad1.15x1.40mm_HandSolder" V 14330 4050 50  0001 C CNN
+F 3 "~" H 14400 4050 50  0001 C CNN
+	1    14400 4050
+	1    0    0    -1
+$EndComp
+$Comp
+L Device:R R2
+U 1 1 5D8E88D9
+P 14150 4050
+F 0 "R2" H 14220 4096 50  0000 L CNN
+F 1 "2.2K" H 14220 4005 50  0000 L CNN
+F 2 "Resistor_SMD:R_0805_2012Metric_Pad1.15x1.40mm_HandSolder" V 14080 4050 50  0001 C CNN
+F 3 "~" H 14150 4050 50  0001 C CNN
+	1    14150 4050
+	1    0    0    -1
+$EndComp
+$Comp
+L Device:R R1
+U 1 1 5D8E893F
+P 13900 4050
+F 0 "R1" H 13970 4096 50  0000 L CNN
+F 1 "2.2K" H 13970 4005 50  0000 L CNN
+F 2 "Resistor_SMD:R_0805_2012Metric_Pad1.15x1.40mm_HandSolder" V 13830 4050 50  0001 C CNN
+F 3 "~" H 13900 4050 50  0001 C CNN
+	1    13900 4050
+	1    0    0    -1
+$EndComp
+$Comp
+L power:+5V #PWR01
+U 1 1 5D8E8A57
+P 13900 3800
+F 0 "#PWR01" H 13900 3650 50  0001 C CNN
+F 1 "+5V" H 13915 3973 50  0000 C CNN
+F 2 "" H 13900 3800 50  0001 C CNN
+F 3 "" H 13900 3800 50  0001 C CNN
+	1    13900 3800
+	1    0    0    -1
+$EndComp
+Wire Wire Line
+	14400 3900 14400 3850
+Wire Wire Line
+	14400 3850 14150 3850
+Wire Wire Line
+	13900 3850 13900 3800
+Wire Wire Line
+	13900 3850 13900 3900
+Connection ~ 13900 3850
+Wire Wire Line
+	14150 3900 14150 3850
+Connection ~ 14150 3850
+Wire Wire Line
+	14150 3850 13900 3850
+Wire Wire Line
+	14400 4300 14400 4200
+Wire Wire Line
+	14400 4300 15100 4300
+Wire Wire Line
+	14150 4400 14150 4200
+Wire Wire Line
+	14150 4400 15100 4400
+Wire Wire Line
+	13900 4500 13900 4200
+Wire Wire Line
+	13900 4500 15100 4500
+$Comp
+L Device:R R8
+U 1 1 5D8EA097
+P 13750 4900
+F 0 "R8" H 13820 4946 50  0000 L CNN
+F 1 "2.2K" H 13820 4855 50  0000 L CNN
+F 2 "Resistor_SMD:R_0805_2012Metric_Pad1.15x1.40mm_HandSolder" V 13680 4900 50  0001 C CNN
+F 3 "~" H 13750 4900 50  0001 C CNN
+	1    13750 4900
+	0    1    1    0
+$EndComp
+$Comp
+L Device:R R9
+U 1 1 5D8EA175
+P 14100 5150
+F 0 "R9" H 14170 5196 50  0000 L CNN
+F 1 "2.2K" H 14170 5105 50  0000 L CNN
+F 2 "Resistor_SMD:R_0805_2012Metric_Pad1.15x1.40mm_HandSolder" V 14030 5150 50  0001 C CNN
+F 3 "~" H 14100 5150 50  0001 C CNN
+	1    14100 5150
+	-1   0    0    1
+$EndComp
+$Comp
+L Device:C C16
+U 1 1 5D8EA2D1
+P 14350 5150
+F 0 "C16" H 14465 5196 50  0000 L CNN
+F 1 "10pF" H 14465 5105 50  0000 L CNN
+F 2 "Capacitor_SMD:C_0805_2012Metric_Pad1.15x1.40mm_HandSolder" H 14388 5000 50  0001 C CNN
+F 3 "~" H 14350 5150 50  0001 C CNN
+	1    14350 5150
+	-1   0    0    1
+$EndComp
+$Comp
+L power:GND #PWR0128
+U 1 1 5D9154FE
+P 14350 5400
+F 0 "#PWR0128" H 14350 5150 50  0001 C CNN
+F 1 "GND" H 14355 5227 50  0000 C CNN
+F 2 "" H 14350 5400 50  0001 C CNN
+F 3 "" H 14350 5400 50  0001 C CNN
+	1    14350 5400
+	1    0    0    -1
+$EndComp
+Wire Wire Line
+	14350 5300 14350 5350
+Wire Wire Line
+	14350 5350 14100 5350
+Wire Wire Line
+	14100 5350 14100 5300
+Connection ~ 14350 5350
+Wire Wire Line
+	14350 5350 14350 5400
+Wire Wire Line
+	13900 4900 14100 4900
+Wire Wire Line
+	14100 4900 14100 5000
+Wire Wire Line
+	14100 4900 14350 4900
+Wire Wire Line
+	14350 4900 14350 5000
+Connection ~ 14100 4900
+Wire Wire Line
+	14350 4900 14650 4900
+Wire Wire Line
+	14650 4900 14650 5100
+Wire Wire Line
+	14650 5100 15500 5100
+Connection ~ 14350 4900
+$Comp
+L power:GND #PWR0129
+U 1 1 5DA770AF
+P 15450 5350
+F 0 "#PWR0129" H 15450 5100 50  0001 C CNN
+F 1 "GND" H 15455 5177 50  0000 C CNN
+F 2 "" H 15450 5350 50  0001 C CNN
+F 3 "" H 15450 5350 50  0001 C CNN
+	1    15450 5350
+	1    0    0    -1
+$EndComp
+Wire Wire Line
+	15450 5200 15450 5350
+Wire Wire Line
+	15450 5200 15500 5200
+$Comp
+L Connector_Generic:Conn_01x02 J4
+U 1 1 5DAFD9E7
+P 15700 5100
+F 0 "J4" H 15780 5092 50  0000 L CNN
+F 1 "Conn_01x02" H 15780 5001 50  0000 L CNN
+F 2 "Connector_PinHeader_2.54mm:PinHeader_1x02_P2.54mm_Vertical" H 15700 5100 50  0001 C CNN
+F 3 "~" H 15700 5100 50  0001 C CNN
+	1    15700 5100
+	1    0    0    -1
+$EndComp
+Wire Wire Line
+	12500 6000 12950 6000
+Text Label 12600 6000 0    50   ~ 0
+DAC_OUT
+Wire Wire Line
+	13150 4900 13600 4900
+Text Label 13200 4900 0    50   ~ 0
+DAC_OUT
 $EndSCHEMATC
