File: 65816/WC65C816_CPU/WC65C816_CPU.kicad_pcb (KiCad board)
At the start: 2 copper layers, 95 x 95 mm, 51 parts, among them J1 USB_B, J2 Conn_01x12, J3 Conn_01x12, J4 Conn_01x02, U1 W65C816S, U2 IS62WV10248EBLL-45TLI, U3 4.9152 MHz, U4 CY8C5267AXI-LP051, U5 MCP23017_SP, U6 AP1117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

Commit message: Added expansion connector
Parts:
- added J5: Conn_02x20_Odd_Even, Connector_PinHeader_2.54mm:PinHeader_2x20_P2.54mm_Vertical, F.Cu at (8.64, 30.5)
Connections:
- U4 pad 24: (no net) -> /~IOINT
- U4 pad 25: (no net) -> /~IOACK
- U4 pad 27: (no net) -> /~IOCS
Routing:
- net /~I2CINT: track 0.00 -> 50.7 mm, vias 0 -> 2
- net /CPUA0: track 0.00 -> 29.2 mm, vias 0 -> 1
- net Net-(U3-Pad8): track 0.00 -> 26.7 mm, vias 0 -> 2
- net /CPUA2: track 0.00 -> 24.5 mm
- net /CPUA1: track 0.00 -> 24.4 mm
- net /CPUA4: track 0.00 -> 21.2 mm
- net /CPUA3: track 0.00 -> 20.3 mm
- net /CPUA6: track 0.00 -> 18.1 mm
- net /CPUA5: track 0.00 -> 16.8 mm
- net /CPUA8: track 0.00 -> 16.5 mm
- net /SCL: track 0.00 -> 16.2 mm
- net /CPUA10: track 0.00 -> 14.5 mm
- net /CPUA7: track 0.00 -> 13.4 mm
- net /CPUA9: track 0.00 -> 12.2 mm
- net /SDA: track 0.00 -> 11.8 mm
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Other:
- board text added: "3.3V A0 A2 A4 A6 A8 A10 A12 A14"
- board text added: "3.3V A1 A3 A5 A7 A9 A11 A13 A15"
- board text added: "D6 D4 D2 D0"
- board text added: "D7 D5 D3 D1"
- board text added: "~CS ~ACK R/~W ~INT"
- board text added: "~RST VPA VPB"
- board text removed: "D4 D3 D5 D6 5V D2 D7"
