File: 65816/WC65C816_CPU/WC65C816_CPU.kicad_pcb (KiCad board)
At the start: 2 copper layers, 95 x 95 mm, 52 parts, among them J1 USB_B, J2 Conn_01x12, J3 Conn_01x12, J4 Conn_01x02, J5 Conn_02x20_Odd_Even, U1 W65C816S, U2 IS62WV10248EBLL-45TLI, U3 4.9152 MHz, U4 CY8C5267AXI-LP051, U5 MCP23017_SP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

Commit message: w65C816
Parts:
- C4, C5: moved to F.Cu
- moved C6 4.23 mm to (62.6, 40.0), turned to 270 degrees
- moved C4 3.75 mm to (71.2, 39.9), turned to 90 degrees
- moved C5 3.30 mm to (69.3, 39.9), turned to 270 degrees
- moved C15 0.77 mm to (27.4, 40.8), turned to 270 degrees
- moved R5 0.25 mm to (88.1, 50.0)
- moved C9 0.25 mm to (88.1, 51.8)
Connections:
- H3 pad 3: /P79 -> /SPISS
- H3 pad 4: /P78 -> /SPISCK
- H3 pad 5: /P77 -> /SPIMOSI
- H3 pad 6: /P76 -> /SPIMISO
- J5 pad 39: (no net) -> GND
- J5 pad 40: (no net) -> GND
- U1 pad 35: /PHI2 -> (no net)
- U2 pad 18: (no net) -> /SRAMA19
- U2 pad 41: /~MEMRD -> (no net)
- U4 pad 1: /R/~W -> /VPA
- U4 pad 23: (no net) -> /~RESB
- U4 pad 3: /~RESB -> /R/~W
- U4 pad 42: (no net) -> /CPUA8
- U4 pad 43: (no net) -> /CPUA9
- U4 pad 69: /CPUA8 -> /SPIMISO
- U4 pad 70: /CPUA9 -> /SPIMOSI
- U4 pad 71: /PHI2 -> /SPISCK
- U4 pad 72: /~MEMRD -> /SPISS
- U4 pad 76: /P76 -> (no net)
- U4 pad 77: /P77 -> (no net)
- U4 pad 78: /P78 -> (no net)
- U4 pad 79: /P79 -> (no net)
- U4 pad 98: /VPB -> /SRAMA19
- U4 pad 99: /VPA -> /VPB
Routing:
- net /CPUA4: track 21.2 -> 45.3 mm, vias 0 -> 2
- net /P79: track 23.4 -> 0.00 mm
- net /P78: track 21.7 -> 0.00 mm
- net /SPISS: track 0.00 -> 19.6 mm
- net /P77: track 19.2 -> 0.00 mm
- net /SPISCK: track 0.00 -> 18.8 mm
- net /CPUA3: track 20.3 -> 38.8 mm, vias 0 -> 2
- net /P76: track 18.3 -> 0.00 mm
- net /CPUA0: track 29.2 -> 47.5 mm, vias 1 -> 3
- net /SPIMOSI: track 0.00 -> 17.9 mm
- net /CPUA2: track 24.5 -> 42.4 mm, vias 0 -> 2
- net /SPIMISO: track 0.00 -> 17.0 mm
- net /CPUA1: track 24.4 -> 40.7 mm, vias 0 -> 2
- net GND: track 30.5 -> 32.0 mm, vias 15 -> 16
- net /~NMI: track 32.8 -> 33.6 mm
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Other:
- board text added: "GND 3.3V SS SCK MOSI MISO"
- board text removed: "GND +V P79 P78 P77 P76"

Commit message: More routing
Parts:
- C6: moved to F.Cu
- moved C5 4.78 mm to (70.2, 35.2), turned to 90 degrees
- moved C16 3.18 mm to (29.8, 62.1)
- moved C4 1.02 mm to (70.4, 39.4)
Connections:
- net Net-(R10-Pad1) renamed /RCS
- net Net-(R7-Pad2) renamed /LED
- J5 pad 32: (no net) -> /VPB
- J5 pad 34: /VPB -> (no net)
- U4 pad 1: /VPA -> (no net)
- U4 pad 48: /~NMI -> (no net)
- U4 pad 6: /CPUA4 -> /SRAMA16
- U4 pad 7: /CPUA5 -> /SRAMA17
- U4 pad 78: (no net) -> /~NMI
- U4 pad 79: (no net) -> /VPA
- U4 pad 8: /CPUA6 -> /SRAMA18
- U4 pad 9: /CPUA7 -> /SRAMA19
- U4 pad 95: /SRAMA16 -> /CPUA4
- U4 pad 96: /SRAMA17 -> /CPUA5
- U4 pad 97: /SRAMA18 -> /CPUA6
- U4 pad 98: /SRAMA19 -> /CPUA7
Routing:
- net /CPUD0: track 21.2 -> 72.0 mm, vias 0 -> 4
- net /CPUD6: track 17.5 -> 68.0 mm, vias 0 -> 2
- net /CPUD7: track 14.3 -> 59.4 mm, vias 0 -> 5
- net /CPUD5: track 14.8 -> 59.8 mm, vias 0 -> 4
- net /CPUD4: track 19.2 -> 61.3 mm, vias 0 -> 4
- net /CPUA11: track 10.5 -> 51.2 mm, vias 0 -> 2
- net /CPUA9: track 12.2 -> 52.5 mm, vias 0 -> 4
- net /VPB: track 0.00 -> 40.3 mm, vias 0 -> 1
- net /CPUA10: track 14.5 -> 54.5 mm, vias 0 -> 4
- net /CPUA14: track 13.5 -> 53.0 mm, vias 0 -> 2
- net /CPUA7: track 13.4 -> 52.6 mm, vias 0 -> 2
- net /CPUA13: track 10.7 -> 49.7 mm, vias 0 -> 2
- net /CPUA12: track 13.9 -> 52.3 mm, vias 0 -> 2
- net /~RESB: track 0.00 -> 36.1 mm, vias 0 -> 1
- net /CPUA6: track 18.1 -> 53.7 mm, vias 0 -> 4
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Other:
- board text added: "~RST VPB"
- board text removed: "~RST VPA VPB"

Commit message: 65c816 card dev
Connections:
- U4 pad 2: /BE -> /CPUA8
- U4 pad 3: /R/~W -> /CPUA9
- U4 pad 42: /CPUA8 -> /R/~W
- U4 pad 43: /CPUA9 -> /BE
