File: 65816/WC65C816_CPU/_autosave-WC65C816_CPU.kicad_pcb (KiCad board)
At the start: 2 copper layers, 95 x 95 mm, 52 parts, among them J1 USB_B, J2 Conn_01x12, J3 Conn_01x12, J4 Conn_01x02, J5 Conn_02x20_Odd_Even, U1 W65C816S, U2 IS62WV10248EBLL-45TLI, U3 4.9152 MHz, U4 CY8C5267AXI-LP051, U5 MCP23017_SP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

Commit message: Switching back to 15 MHz to run zexall
Parts:
- C4, C5: moved to F.Cu
- moved C4 5.75 mm to (78.7, 42.5)
- moved C6 4.23 mm to (62.6, 40.0), turned to 270 degrees
- moved C5 3.30 mm to (69.3, 39.9), turned to 270 degrees
- moved C15 0.77 mm to (27.4, 40.8), turned to 270 degrees
- moved R5 0.25 mm to (88.1, 50.0)
- moved C9 0.25 mm to (88.1, 51.8)
Connections:
- H3 pad 3: /P79 -> /SPISS
- H3 pad 4: /P78 -> /SPISCK
- H3 pad 5: /P77 -> /SPIMOSI
- H3 pad 6: /P76 -> /SPIMISO
- J5 pad 39: (no net) -> GND
- J5 pad 40: (no net) -> GND
- U1 pad 35: /PHI2 -> (no net)
- U2 pad 18: (no net) -> /SRAMA19
- U2 pad 41: /~MEMRD -> (no net)
- U4 pad 1: /R/~W -> /VPA
- U4 pad 23: (no net) -> /~RESB
- U4 pad 3: /~RESB -> /R/~W
- U4 pad 42: (no net) -> /CPUA8
- U4 pad 43: (no net) -> /CPUA9
- U4 pad 69: /CPUA8 -> /SPIMISO
- U4 pad 70: /CPUA9 -> /SPIMOSI
- U4 pad 71: /PHI2 -> /SPISCK
- U4 pad 72: /~MEMRD -> /SPISS
- U4 pad 76: /P76 -> (no net)
- U4 pad 77: /P77 -> (no net)
- U4 pad 78: /P78 -> (no net)
- U4 pad 79: /P79 -> (no net)
- U4 pad 98: /VPB -> /SRAMA19
- U4 pad 99: /VPA -> /VPB
Routing:
- net /CPUA4: track 21.2 -> 44.9 mm, vias 0 -> 2
- net /P79: track 23.4 -> 0.00 mm
- net /P78: track 21.7 -> 0.00 mm
- net /SPISS: track 0.00 -> 19.6 mm
- net /P77: track 19.2 -> 0.00 mm
- net /SPISCK: track 0.00 -> 18.8 mm
- net /P76: track 18.3 -> 0.00 mm
- net /SPIMOSI: track 0.00 -> 17.9 mm
- net /SPIMISO: track 0.00 -> 17.0 mm
- net /CPUA3: track 20.3 -> 21.6 mm
- net /~I2CINT: track 50.7 -> 51.4 mm
Other:
- board text added: "GND +3.3V SS SCK MOSI MISO"
- board text removed: "GND +V P79 P78 P77 P76"
