File: 65816/WC65C816_CPU/WC65C816_CPU.sch (KiCad schematic (older format))
At the start: 51 parts, among them J1 USB_B, J2 Conn_01x12, J3 Conn_01x12, J4 Conn_01x02, U1 W65C816S, U2 IS62WV10248EBLL-45TLI, U3 4.9152 MHz, U4 CY8C5267AXI-LP051, U5 MCP23017_SP, U6 AP1117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

Commit message: Added expansion connector
Parts:
- added J5: Conn_02x20_Odd_Even, Connector_PinHeader_2.54mm:PinHeader_2x20_P2.54mm_Vertical, symbol Connector_Generic:Conn_02x20_Odd_Even
Connections:
- net labels added: ~IOACK, ~IOCS, ~IOINT
- wire segments 394 -> 440
- no-connect marks 15 -> 13
Other:
- note added: "CPU BUS EXPANDER"
- moved on the sheet: J2, J3, U5

Commit message: Switching back to 15 MHz to run zexall
Parts:
- MTG1, MTG2, MTG3, MTG4: symbol LandBoards:MTG_HOLE -> WC65C816_CPU-rescue:MTG_HOLE-LandBoards
- U1: symbol LandBoards_Semis:W65C816S -> WC65C816_CPU-rescue:W65C816S-LandBoards_Semis
- U2: symbol LandBoards_Semis:IS62WV10248EBLL-45TLI -> WC65C816_CPU-rescue:IS62WV10248EBLL-45TLI-LandBoards_Semis
- U3: symbol LandBoards_Semis:OSC -> WC65C816_CPU-rescue:OSC-LandBoards_Semis
- U4: symbol LandBoards_Semis:CY8C5888AXI-LP096 -> WC65C816_CPU-rescue:CY8C5888AXI-LP096-LandBoards_Semis
- U6: symbol LandBoards_Semis:AP1117 -> WC65C816_CPU-rescue:AP1117-LandBoards_Semis
Connections:
- net labels added: SPIMISO, SPIMOSI, SPISCK, SPISS, SRAMA19
- wire segments 440 -> 445
Other:
- note added: "MISO\nMOSI\nSCK\nSS\n+3.3V\nGND"
- moved on the sheet: J5
Changed lines of the file:
@@
 Wire Wire Line
 	9300 6950 9900 6950
-Text Label 9400 7650 0    50   ~ 0
+Text Label 12600 6750 0    50   ~ 0
 CPUA8
 Wire Wire Line
 	9300 7050 9900 7050
-Text Label 9400 7550 0    50   ~ 0
+Text Label 12600 6650 0    50   ~ 0
 CPUA9
 Wire Wire Line
@@
 Text Label 9400 7250 0    50   ~ 0
 CPUA12
-Wire Wire Line
-	9300 7450 9900 7450
 Text Label 9400 7150 0    50   ~ 0
 CPUA13
@@
 Text Label 9400 3850 0    50   ~ 0
 ~MEMWR
-Text Label 9400 3950 0    50   ~ 0
+Text Label 8150 4000 0    50   ~ 0
 ~MEMRD
 Wire Wire Line
@@
 Text Label 5000 1400 0    50   ~ 0
 ~RESB
-Text Label 9400 5250 0    50   ~ 0
+Text Label 9400 4650 0    50   ~ 0
 ~RESB
 Wire Wire Line
-	9300 5250 9900 5250
+	9300 4650 9900 4650
 Wire Wire Line
 	9300 6350 9900 6350
@@
 	9300 6750 9900 6750
 Wire Wire Line
+	9300 5350 9900 5350
+Wire Wire Line
 	9300 5450 9900 5450
-Wire Wire Line
-	9300 5550 9900 5550
 $Comp
 L power:GND #PWR0106
@@
 Text Label 5000 1700 0    50   ~ 0
 PHI2
-Text Label 9400 4050 0    50   ~ 0
+Text Label 8150 4100 0    50   ~ 0
 PHI2
 Text Label 5000 2000 0    50   ~ 0
@@
 Text Label 9400 6150 0    50   ~ 0
 MX
-Text Label 9400 5350 0    50   ~ 0
+Text Label 9400 5250 0    50   ~ 0
 R/~W
 Text Label 9400 6250 0    50   ~ 0
 VDA
+Text Label 9400 5350 0    50   ~ 0
+VPA
 Text Label 9400 5450 0    50   ~ 0
-VPA
-Text Label 9400 5550 0    50   ~ 0
 VPB
 Wire Wire Line
@@
 	12450 5550 13050 5550
 Wire Wire Line
-	9300 5350 9900 5350
+	9300 5250 9900 5250
 $Comp
 L Device:LED_Small_ALT D1
@@
 $EndComp
 $Comp
-L LandBoards_Semis:OSC U3
+L WC65C816_CPU-rescue:OSC-LandBoards_Semis U3
 U 1 1 5E0B1D6E
 P 13750 7300
@@
 	11950 1300 12150 1300
 $Comp
-L LandBoards_Semis:CY8C5888AXI-LP096 U4
+L WC65C816_CPU-rescue:CY8C5888AXI-LP096-LandBoards_Semis U4
 U 1 1 5D746915
 P 11250 5200
@@
 	9900 4250 8950 4250
 $Comp
-L LandBoards:MTG_HOLE MTG4
+L WC65C816_CPU-rescue:MTG_HOLE-LandBoards MTG4
 U 1 1 5E2D4C5F
 P 11200 10350
@@
 $EndComp
 $Comp
-L LandBoards:MTG_HOLE MTG3
+L WC65C816_CPU-rescue:MTG_HOLE-LandBoards MTG3
 U 1 1 5E2D5046
 P 10200 10350
@@
 $EndComp
 $Comp
-L LandBoards:MTG_HOLE MTG2
+L WC65C816_CPU-rescue:MTG_HOLE-LandBoards MTG2
 U 1 1 5E2D50A8
 P 9200 10350
@@
 $EndComp
 $Comp
-L LandBoards:MTG_HOLE MTG1
+L WC65C816_CPU-rescue:MTG_HOLE-LandBoards MTG1
 U 1 1 5E2D5139
 P 8200 10350
@@
 Wire Wire Line
 	13850 1950 14450 1950
-Text Label 14000 1950 0    50   ~ 0
-P78
-Text Label 14000 1850 0    50   ~ 0
-P77
+Text Label 9400 4050 0    50   ~ 0
+SPISCK
+Text Label 9400 7550 0    50   ~ 0
+SPIMOSI
 Wire Wire Line
 	13850 1750 14450 1750
 Wire Wire Line
 	13850 2050 14450 2050
-Text Label 14000 2050 0    50   ~ 0
-P79
-Text Label 14000 1750 0    50   ~ 0
-P76
+Text Label 9400 3950 0    50   ~ 0
+SPISS
+Text Label 9400 7650 0    50   ~ 0
+SPIMISO
 $Comp
 L Connector_Generic:Conn_01x06 H3
@@
 NoConn ~ 9900 4750
 $Comp
-L LandBoards_Semis:W65C816S U1
+L WC65C816_CPU-rescue:W65C816S-LandBoards_Semis U1
 U 1 1 5DABCA35
 P 6200 2600
@@
 BE
 $Comp
-L LandBoards_Semis:IS62WV10248EBLL-45TLI U2
+L WC65C816_CPU-rescue:IS62WV10248EBLL-45TLI-LandBoards_Semis U2
 U 1 1 5DFB44A5
 P 6250 6500
@@
 $EndComp
 $Comp
-L LandBoards_Semis:AP1117 U6
+L WC65C816_CPU-rescue:AP1117-LandBoards_Semis U6
 U 1 1 5E1BB45D
 P 5600 9650
@@
 L Connector_Generic:Conn_02x20_Odd_Even J5
 U 1 1 5DAB55CC
-P 2650 2150
-F 0 "J5" H 2750 3150 50  0000 C CNN
-F 1 "Conn_02x20_Odd_Even" H 2700 1050 50  0000 C CNN
-F 2 "Connector_PinHeader_2.54mm:PinHeader_2x20_P2.54mm_Vertical" H 2600 950 50  0000 C CNN
-F 3 "~" H 2650 2150 50  0001 C CNN
-	1    2650 2150
+P 2650 2050
+F 0 "J5" H 2750 3050 50  0000 C CNN
+F 1 "Conn_02x20_Odd_Even" H 2700 950 50  0000 C CNN
+F 2 "Connector_PinHeader_2.54mm:PinHeader_2x20_P2.54mm_Vertical" H 2600 850 50  0000 C CNN
+F 3 "~" H 2650 2050 50  0001 C CNN
+	1    2650 2050
 	1    0    0    -1
 $EndComp
@@
 CPUA15
 Wire Wire Line
-	2250 1250 2250 1100
+	2250 1150 2250 1000
 $Comp
 L power:+3.3V #PWR02
 U 1 1 5DB8380B
-P 2250 1000
-F 0 "#PWR02" H 2250 850 50  0001 C CNN
-F 1 "+3.3V" H 2265 1173 50  0000 C CNN
-F 2 "" H 2250 1000 50  0001 C CNN
-F 3 "" H 2250 1000 50  0001 C CNN
-	1    2250 1000
-	1    0    0    -1
-$EndComp
-Wire Wire Line
-	2250 1250 2450 1250
+P 2250 900
+F 0 "#PWR02" H 2250 750 50  0001 C CNN
+F 1 "+3.3V" H 2265 1073 50  0000 C CNN
+F 2 "" H 2250 900 50  0001 C CNN
+F 3 "" H 2250 900 50  0001 C CNN
+	1    2250 900
+	1    0    0    -1
+$EndComp
+Wire Wire Line
+	2250 1150 2450 1150
 Wire Wire Line
 	1850 2450 2450 2450
@@
 CPUD7
 Wire Wire Line
-	2250 1100 3050 1100
-Wire Wire Line
-	3050 1100 3050 1250
-Wire Wire Line
-	3050 1250 2950 1250
-Connection ~ 2250 1100
-Wire Wire Line
-	2250 1100 2250 1000
-Wire Wire Line
-	2450 3150 2150 3150
-Wire Wire Line
-	2150 3150 2150 3400
-Wire Wire Line
-	2150 3400 3200 3400
-Wire Wire Line
-	3200 3400 3200 3150
-Wire Wire Line
-	3200 3150 2950 3150
-Connection ~ 2150 3400
-Wire Wire Line
-	2150 3400 2150 3550
+	2250 1000 3050 1000
+Wire Wire Line
+	3050 1000 3050 1150
+Wire Wire Line
+	3050 1150 2950 1150
+Connection ~ 2250 1000
+Wire Wire Line
+	2250 1000 2250 900
+Wire Wire Line
+	2450 3050 2150 3050
+Wire Wire Line
+	2150 3050 2150 3300
+Wire Wire Line
+	2150 3300 3200 3300
+Wire Wire Line
+	3200 3300 3200 3050
+Wire Wire Line
+	3200 3050 2950 3050
+Connection ~ 2150 3300
+Wire Wire Line
+	2150 3300 2150 3450
 $Comp
 L power:GND #PWR01
 U 1 1 5E2C1042
-P 2150 3550
-F 0 "#PWR01" H 2150 3300 50  0001 C CNN
-F 1 "GND" H 2155 3377 50  0000 C CNN
-F 2 "" H 2150 3550 50  0001 C CNN
-F 3 "" H 2150 3550 50  0001 C CNN
-	1    2150 3550
+P 2150 3450
+F 0 "#PWR01" H 2150 3200 50  0001 C CNN
+F 1 "GND" H 2155 3277 50  0000 C CNN
+F 2 "" H 2150 3450 50  0001 C CNN
+F 3 "" H 2150 3450 50  0001 C CNN
+	1    2150 3450
 	1    0    0    -1
 $EndComp
@@
 	1850 2750 2450 2750
 Wire Wire Line
-	2950 2650 3550 2650
-Text Label 3150 2650 0    50   ~ 0
+	2950 1250 3550 1250
+Text Label 3150 1250 0    50   ~ 0
 VPA
 Wire Wire Line
@@
 Wire Wire Line
 	1850 2850 2450 2850
+Wire Wire Line
+	1850 1250 2450 1250
+Text Label 1950 1250 0    50   ~ 0
+~NMI
+Wire Wire Line
+	5050 7300 5650 7300
+Text Label 5150 7300 0    50   ~ 0
+SRAMA19
+Wire Wire Line
+	9300 5550 9900 5550
+Text Label 9400 5550 0    50   ~ 0
+SRAMA19
+Text Notes 14700 2300 0    63   ~ 0
+MISO\nMOSI\nSCK\nSS\n+3.3V\nGND
+Text Label 13950 1950 0    50   ~ 0
+SPISCK
+Text Label 13950 1850 0    50   ~ 0
+SPIMOSI
+Text Label 13950 2050 0    50   ~ 0
+SPISS
+Text Label 13950 1750 0    50   ~ 0
+SPIMISO
+Wire Wire Line
+	9300 7450 9900 7450
+Wire Wire Line
+	12450 6750 13050 6750
+Wire Wire Line
+	12450 6650 13050 6650
 $EndSCHEMATC

Commit message: More routing
Connections:
- net labels added: LED, RCS
Other:
- moved on the sheet: R10
Changed lines of the file:
@@
 CPUD7
 Wire Wire Line
-	12450 4250 13050 4250
+	9300 5550 9900 5550
 Text Label 12550 4950 0    50   ~ 0
 CPUA0
 Wire Wire Line
-	12450 4350 13050 4350
+	9300 5650 9900 5650
 Text Label 12550 4850 0    50   ~ 0
 CPUA1
 Wire Wire Line
-	12450 4450 13050 4450
+	9300 5750 9900 5750
 Text Label 12550 4750 0    50   ~ 0
 CPUA2
 Wire Wire Line
-	12450 4550 13050 4550
+	9300 5850 9900 5850
 Text Label 12550 4650 0    50   ~ 0
 CPUA3
 Wire Wire Line
 	12450 4650 13050 4650
-Text Label 12550 4550 0    50   ~ 0
+Text Label 9400 5850 0    50   ~ 0
 CPUA4
 Wire Wire Line
 	12450 4750 13050 4750
-Text Label 12550 4450 0    50   ~ 0
+Text Label 9400 5750 0    50   ~ 0
 CPUA5
 Wire Wire Line
 	12450 4850 13050 4850
-Text Label 12550 4350 0    50   ~ 0
+Text Label 9400 5650 0    50   ~ 0
 CPUA6
 Wire Wire Line
 	12450 4950 13050 4950
-Text Label 12550 4250 0    50   ~ 0
+Text Label 9400 5550 0    50   ~ 0
 CPUA7
 Wire Wire Line
@@
 	9300 4650 9900 4650
 Wire Wire Line
-	9300 6350 9900 6350
+	9300 3450 9900 3450
 Wire Wire Line
 	9300 6450 9900 6450
@@
 	9300 6750 9900 6750
 Wire Wire Line
-	9300 5350 9900 5350
+	9300 3350 9900 3350
 Wire Wire Line
 	9300 5450 9900 5450
@@
 Text Label 5000 2100 0    50   ~ 0
 ~IRQ
-Text Label 9400 6350 0    50   ~ 0
+Text Label 9400 3450 0    50   ~ 0
 ~NMI
 Text Label 9400 6450 0    50   ~ 0
@@
 Text Label 9400 6250 0    50   ~ 0
 VDA
-Text Label 9400 5350 0    50   ~ 0
+Text Label 9400 3350 0    50   ~ 0
 VPA
 Text Label 9400 5450 0    50   ~ 0
@@
 	9300 6150 9900 6150
 Wire Wire Line
-	9300 5650 9900 5650
+	12450 4350 13050 4350
 Wire Wire Line
 	12450 5550 13050 5550
@@
 Connection ~ 11350 1300
 Wire Wire Line
-	9300 5750 9900 5750
-Wire Wire Line
-	9300 5850 9900 5850
+	12450 4450 13050 4450
+Wire Wire Line
+	12450 4550 13050 4550
 Wire Wire Line
 	5050 5400 5650 5400
@@
 Text Label 5150 7200 0    50   ~ 0
 SRAMA18
-Text Label 9400 5850 0    50   ~ 0
+Text Label 12550 4550 0    50   ~ 0
 SRAMA16
-Text Label 9400 5750 0    50   ~ 0
+Text Label 12550 4450 0    50   ~ 0
 SRAMA17
-Text Label 9400 5650 0    50   ~ 0
+Text Label 12550 4350 0    50   ~ 0
 SRAMA18
 Text Label 12600 5350 0    50   ~ 0
@@
 SWD
 Wire Wire Line
-	9300 3450 9900 3450
+	9300 6350 9900 6350
 Wire Wire Line
 	9300 3550 9900 3550
-Text Label 9400 3450 0    50   ~ 0
+Text Label 9400 6350 0    50   ~ 0
 P78
 Text Label 9400 3550 0    50   ~ 0
 P77
 Wire Wire Line
-	9300 3350 9900 3350
+	9300 5350 9900 5350
 Wire Wire Line
 	9300 3650 9900 3650
-Text Label 9400 3350 0    50   ~ 0
+Text Label 9400 5350 0    50   ~ 0
 P79
 Text Label 9400 3650 0    50   ~ 0
@@
 L Device:R R10
 U 1 1 5E156E10
-P 5350 8000
-F 0 "R10" V 5250 7950 50  0000 L CNN
-F 1 "2.2K" V 5450 7950 50  0000 L CNN
-F 2 "Resistor_SMD:R_0805_2012Metric_Pad1.15x1.40mm_HandSolder" V 5280 8000 50  0001 C CNN
-F 3 "~" H 5350 8000 50  0001 C CNN
-	1    5350 8000
+P 5150 8000
+F 0 "R10" V 5050 7950 50  0000 L CNN
+F 1 "2.2K" V 5250 7950 50  0000 L CNN
+F 2 "Resistor_SMD:R_0805_2012Metric_Pad1.15x1.40mm_HandSolder" V 5080 8000 50  0001 C CNN
+F 3 "~" H 5150 8000 50  0001 C CNN
+	1    5150 8000
 	0    1    1    0
 $EndComp
@@
 	5600 7600 5600 8000
 Wire Wire Line
-	5600 8000 5500 8000
-Wire Wire Line
-	5200 8000 4950 8000
+	5600 8000 5300 8000
+Wire Wire Line
+	5000 8000 4950 8000
 $Comp
 L power:+3.3V #PWR0102
@@
 VPA
 Wire Wire Line
-	2950 2750 3550 2750
-Text Label 3150 2750 0    50   ~ 0
+	2950 2650 3550 2650
+Text Label 3150 2650 0    50   ~ 0
 VPB
 Text Label 9400 4550 0    50   ~ 0
@@
 SRAMA19
 Wire Wire Line
-	9300 5550 9900 5550
-Text Label 9400 5550 0    50   ~ 0
+	12450 4250 13050 4250
+Text Label 12550 4250 0    50   ~ 0
 SRAMA19
 Text Notes 14700 2300 0    63   ~ 0
@@
 Wire Wire Line
 	12450 6650 13050 6650
+Text Label 9400 4250 0    50   ~ 0
+LED
+Text Label 5400 8000 0    50   ~ 0
+RCS
 $EndSCHEMATC

Commit message: 65c816 card dev
Changed lines of the file:
@@
 EESchema Schematic File Version 4
-LIBS:WC65C816_CPU-cache
-EELAYER 26 0
+EELAYER 30 0
 EELAYER END
 $Descr B 17000 11000
@@
 Wire Wire Line
 	9300 6950 9900 6950
-Text Label 12600 6750 0    50   ~ 0
+Text Label 9400 5150 0    50   ~ 0
 CPUA8
 Wire Wire Line
 	9300 7050 9900 7050
-Text Label 12600 6650 0    50   ~ 0
+Text Label 9400 5250 0    50   ~ 0
 CPUA9
 Wire Wire Line
@@
 Text Label 9400 6150 0    50   ~ 0
 MX
-Text Label 9400 5250 0    50   ~ 0
+Text Label 12600 6750 0    50   ~ 0
 R/~W
 Text Label 9400 6250 0    50   ~ 0
@@
 Wire Wire Line
 	9300 5150 9900 5150
-Text Label 9400 5150 0    50   ~ 0
+Text Label 12600 6650 0    50   ~ 0
 BE
 $Comp
