File: Z80/Z80_PCB_Design/FrontPanel/FrontPanel.sch (KiCad schematic (older format))
At the start: 116 parts, among them J1 Conn_01x02, J2 CONN_4, J3 CONN_4, J6 CONN_02X02, SW1 SW_Push, SW10 SW_Push, SW11 SW_Push, SW12 SW_Push, SW13 SW_Push, SW14 SW_Push, SW15 SW_Push, SW16 SW_Push, SW17 SW_Push, SW18 SW_Push, SW19 SW_Push, SW2 SW_Push, SW20 SW_Push, SW21 SW_Push, SW22 SW_Push, SW23 SW_Push, SW24 SW_Push, SW25 SW_Push, SW26 SW_Push, SW27 SW_Push, SW28 SW_Push, SW29 SW_Push, SW3 SW_Push, SW30 SW_Push, SW31 SW_Push, SW32 SW_Push, SW4 SW_Push, SW5 SW_Push, SW6 SW_Push, SW7 SW_Push, SW8 SW_Push, SW9 SW_Push, U1 MCP23017-E/SS, U2 MCP23017-E/SS, U3 MCP23017-E/SS, U4 MCP23017-E/SS

Commit message: Added I2C interface to Z80 CPU
Parts:
- removed J2: CONN_4, Connector_PinHeader_2.54mm:PinHeader_1x04_P2.54mm_Vertical, symbol FrontPanel-rescue:CONN_4
- removed ST1: CONN_1, symbol FrontPanel-rescue:CONN_1
- added J2: Conn_01x05, Connector_PinHeader_2.54mm:PinHeader_1x05_P2.54mm_Vertical, symbol Connector_Generic:Conn_01x05
- R10, R11, R12, R13, R14, R15, R16, R17, R18, R19, R20, R21, R22, R23, R24, R25, R26, R27, R28, R29, R30, R31, R32, R33, R34, R35, R36, R37, R38, R5, R8, R9: value 330 -> 560
- TEST1: renamed from ST2; footprint (none) -> LandBoards_Marking:TEST_BLK-REAR
Connections:
- wire segments 363 -> 371
- no-connect marks 2 -> 1
Other:
- note added: "CARD I2C\nA2 Address\nSelect"
- note added: "CONFIGURATION AND PROGRAMMING NOTES:\n1 - SWITCHES NEED TO BE PULLED UP BY THE INTERNAL PULL UP RESISTORS IN THE MCP23017 PARTS.\n2 - INTA AND INTB NEED TO BE CONFIGURED AS OPEN-DRAIN OUTPUTS. THEY ARE PULLED UP ON THIS BOARD.\n3 - THE HOST SOFTWARE CAN RUN IN INTERRUPT DRIVEN MODE BUT WILL NEED TO POLL THE CHIPS TO DETERMINE THE INTERRUPT SOURCE.\n4 - SWITCHES ARE ON A-PORTS. PULL-UP RESISTORS M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"
- note added: "I2C Connectors\n(Daisy-chain)"
- note added: "I2C Terminators"
- note added: "~INT\nSCL\nSDA\nVCC\nGND"
- moved on the sheet: DS1, DS10, DS11, DS12, DS13, DS14, DS15, DS16, DS17, DS18, DS19, DS2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

Commit message: PSoC Front panel WIP
Other:
- note added: "ADDRESS = 0x24\n(TOP ROW)"
- note added: "ADDRESS = 0x25\n(2nd ROW DOWN)"
- note added: "ADDRESS = 0x26\n(3rd ROW DOWN)"
- note added: "ADDRESS = 0x27\n(BOTTOM ROW)"
Changed lines of the file:
@@
 	2150 3500 2150 3850
 Connection ~ 2150 3850
-Text Notes 1100 1900 0    50   ~ 0
+Text Notes 950  2550 0    100  Italic 20
 CARD I2C\nA2 Address\nSelect
 Text Notes 3550 4000 2    50   ~ 0
 I2C Terminators
-Text Notes 1150 4850 0    50   ~ 0
+Text Notes 850  5200 0    100  Italic 20
 I2C Connectors\n(Daisy-chain)
 Wire Wire Line
@@
 Wire Wire Line
 	1700 3550 2350 3550
+Text Notes 13150 4850 0    100  Italic 20
+ADDRESS = 0x24\n(TOP ROW)
+Text Notes 10550 4900 0    100  Italic 20
+ADDRESS = 0x25\n(2nd ROW DOWN)
+Text Notes 7900 4900 0    100  Italic 20
+ADDRESS = 0x26\n(3rd ROW DOWN)
+Text Notes 5300 4850 0    100  Italic 20
+ADDRESS = 0x27\n(BOTTOM ROW)
 $EndSCHEMATC

Commit message: pio init stuck z80
Parts:
- U1, U2, U3, U4: symbol LandBoards_Semis:MCP23017P -> FrontPanel-rescue:MCP23017P-LandBoards_Semis
Changed lines of the file:
@@
 Connection ~ 7250 4550
 $Comp
-L LandBoards_Semis:MCP23017P U1
+L FrontPanel-rescue:MCP23017P-LandBoards_Semis U1
 U 1 1 5DC44742
 P 5300 3000
@@
 $EndComp
 $Comp
-L LandBoards_Semis:MCP23017P U2
+L FrontPanel-rescue:MCP23017P-LandBoards_Semis U2
 U 1 1 5DC44E1C
 P 7950 3000
@@
 $EndComp
 $Comp
-L LandBoards_Semis:MCP23017P U3
+L FrontPanel-rescue:MCP23017P-LandBoards_Semis U3
 U 1 1 5DC44F08
 P 10500 3000
@@
 $EndComp
 $Comp
-L LandBoards_Semis:MCP23017P U4
+L FrontPanel-rescue:MCP23017P-LandBoards_Semis U4
 U 1 1 5DC45000
 P 13050 3000
